File: Hardware/ichos.kicad_sch (KiCad schematic)
At the start: 21 parts, among them J1 629722000214, U1 XU316-1024-QF60B-C24, U2 W25Q80EWSNIG, Y1 24.0MHz

Commit message: update
Parts:
- removed C1, C2: 16pF, Capacitor_SMD:C_0402_1005Metric, symbol Device:C_Small
- removed C3, C4: 100nF, Capacitor_SMD:C_0402_1005Metric, symbol Device:C_Small
- removed R1: 1M, Resistor_SMD:R_0402_1005Metric, symbol Device:R_Small
- removed R2: 680R, Resistor_SMD:R_0402_1005Metric, symbol Device:R_Small
- removed R3: 4K7, Resistor_SMD:R_0402_1005Metric, symbol Device:R_Small
- removed R4: 10K, Resistor_SMD:R_0402_1005Metric, symbol Device:R_Small
- removed S1: 430481031816, ichos:430481031816, symbol ichos:430481031816
- removed U1: XU316-1024-QF60B-C24, QFN_F60B-C24_XMO, symbol ichos:XU316-1024-QF60B-C24
- removed U2: W25Q80EWSNIG, Package_SO:SOIC-8_5.23x5.23mm_P1.27mm, symbol Memory_Flash:W25Q16JVSS
- removed Y1: 24.0MHz, ichos:830108340709, symbol Device:Crystal_GND23
- R5, R6, R7: Rating %1 -> 1%
Other:
- added sheet MCU (MCU.kicad_sch)
- added sheet Power (Power.kicad_sch)
- note removed: "CRYSTAL"
- note removed: "QSPI FLASH"
- note removed: "RESET"
- moved on the sheet: C5, C6, D1, F1, FL1, J1, R5, R6, R7

Commit message: power
Parts:
- removed D1: SKM14, Diode_SMD:D_SOD-123F, symbol Device:D_Schottky
- removed F1: 0ZCG0035FF2C, Fuse:Fuse_1812_4532Metric, symbol Device:Polyfuse
Connections:
- net at C5.2, J1.S1 (SHIELD), R5.2: no longer J1.S2 (SHIELD2), J1.S3 (SHIELD2), J1.S4 (SHIELD2)
Other:
- added sheet Amplifier (Amplifier.kicad_sch)
- moved on the sheet: C5, C6, FL1, J1, R5, R6, R7
